File: coco3/coco3.kicad_pcb (KiCad board)
At the start: 2 copper layers, 280 x 155.3 mm, 218 parts, among them CN1 Conn_02x20_Odd_Even, CN2 Conn_01x16_Female, CN3 Conn_02x05_Odd_Even, CN4 Conn_01x12_Female, CN5 Conn_01x12_Female, CN6 Conn_01x12_Female, CN7 Conn_01x03_Male, IC1 MC6809E, IC10 74LS244, IC11 74LS244, IC12 74LS244, IC13 74LS374, IC14 74LS30, IC15 74LS04, IC16 TMS4464, IC17 TMS4464, IC18 TMS4464, IC19 TMS4464, IC2 27C256, IC3 SN74LS245N, IC36 MC78L08_TO92, IC4 W65C21N6TPG-14, IC5 W65C21N6TPG-14, IC6 TCC1014, IC7 SC77526, IC8 SC77527P, IC9 74LS138, J5A1001 CVIDEO, J5B1001 SOUND, Q1 2N6123, Q2 2SC945(NTE85), Q3 2SC945(NTE85), Q4 MPSA13(NTE46), Q5 2SC945(NTE85), Q6 2SC945(NTE85), Q7 2SC945(NTE85), SW1 SW_DPDT_x2, SW2 Reset Switch, SW3 SW3, X1 28.63636 MHz

Commit message: changed title to CoCo++ and changed revision to 1.0.0
Other:
- board text added: "CoCo++"
- board text added: "Rev. 1.0.0"
- board text removed: "ATHENA"
- board text removed: "Rev. 1.1.0"
Changed lines of the file:
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@@
   (general
     (thickness 1.6)
-    (drawings 139)
+    (drawings 138)
     (tracks 5367)
     (zones 0)
@@
   (page USLegal)
   (title_block
-    (title "TRS-80 Color Computer 3")
-    (date 2021-03-24)
-    (rev 1.1.0)
-    (comment 3 "This PCB is based on ")
+    (title CoCo++)
+    (date 2021-08-31)
+    (rev 1.0.0)
     (comment 4 "Rocky Hill")
   )
   (layers
-    (0 F.Cu signal)
-    (31 B.Cu signal)
+    (0 F.Cu signal hide)
+    (31 B.Cu signal hide)
     (32 B.Adhes user)
     (33 F.Adhes user)
@@
     (effects (font (size 1 1) (thickness 0.15)))
   )
-  (gr_text "Rev. 1.1.0" (at 307.0014 168.074) (layer F.SilkS)
+  (gr_text "Rev. 1.0.0" (at 307.0014 168.074) (layer F.SilkS)
     (effects (font (size 1.5 1.5) (thickness 0.3)))
   )
@@
     (effects (font (size 1 1) (thickness 0.15)) (justify left))
   )
-  (gr_text "Rev. 1.1.0" (at 187.8514 114.624) (layer F.SilkS)
-    (effects (font (size 1.5 1.5) (thickness 0.3)))
-  )
-  (gr_text "ATHENA " (at 172.5014 114.074) (layer F.SilkS)
+  (gr_text CoCo++ (at 172.5014 114.074) (layer F.SilkS)
     (effects (font (size 3 3) (thickness 0.6)))
   )
