File: coco3/coco3.kicad_pcb (KiCad board)
At the start: 2 copper layers, 280 x 155.3 mm, 218 parts, among them CN1 Conn_02x20_Odd_Even, CN2 Conn_01x16_Female, CN3 Conn_02x05_Odd_Even, CN4 Conn_01x12_Female, CN5 Conn_01x12_Female, CN6 Conn_01x12_Female, CN7 Conn_01x03_Male, IC1 MC6809E, IC10 74LS244, IC11 74LS244, IC12 74LS244, IC13 74LS374, IC14 74LS30, IC15 74LS04, IC16 TMS4464, IC17 TMS4464, IC18 TMS4464, IC19 TMS4464, IC2 27C256, IC3 SN74LS245N, IC36 MC78L08_TO92, IC4 W65C21N6TPG-14, IC5 W65C21N6TPG-14, IC6 TCC1014, IC7 SC77526, IC8 SC77527P, IC9 74LS138, J5A1001 CVIDEO, J5B1001 SOUND, Q1 2N6123, Q2 2SC945(NTE85), Q3 2SC945(NTE85), Q4 MPSA13(NTE46), Q5 2SC945(NTE85), Q6 2SC945(NTE85), Q7 2SC945(NTE85), SW1 SW_DPDT_x2, SW2 Reset Switch, SW3 SW3, X1 28.63636 MHz

Commit message: -replaced PIA's with he PLCC44 package versions -removed RF modulator -removed DRAM
Parts:
- removed C43, C44, C45, C46: .1uF, Capacitor_THT:C_Disc_D4.7mm_W2.5mm_P5.00mm
- removed C65: 82pF, Capacitor_THT:C_Rect_L7.2mm_W3.0mm_P5.00mm_FKS2_FKP2_MKS2_MKP2
- removed C66: 27pF, Capacitor_THT:C_Rect_L7.2mm_W3.0mm_P5.00mm_FKS2_FKP2_MKS2_MKP2
- removed C67: 10uF 25v, Capacitor_THT:CP_Radial_D5.0mm_P2.00mm
- removed IC16, IC17, IC18, IC19: TMS4464, Package_DIP:DIP-18_W7.62mm_Socket
- removed JP65, JP66: SolderJumper_2_Open, Jumper:SolderJumper-2_P1.3mm_Open_RoundedPad1.0x1.5mm
- removed R26: 2.2K, Resistor_THT:R_Axial_DIN0207_L6.3mm_D2.5mm_P10.16mm_Horizontal
- removed R60: 100, Resistor_THT:R_Axial_DIN0207_L6.3mm_D2.5mm_P10.16mm_Horizontal
- removed REF1: OSHW-Logo2_9.8x8mm_SilkScreen, Symbol:OSHW-Logo2_9.8x8mm_SilkScreen
- removed REF2: OSHW-Logo2_14.6x12mm_SilkScreen, Symbol:OSHW-Logo2_14.6x12mm_SilkScreen
- removed RF1: CoCo3RFModulator, coco2:CoCo 3 RF Modulator
- removed SW3: SW3, coco2:SW_EG1213
- IC4, IC5: value W65C21N6TPG-14 -> W65C21N6TPLG-14; footprint Package_DIP:DIP-40_W15.24mm_Socket -> Package_LCC:PLCC-44_THT-Socket
- moved IC4 52.3 mm to (128.4, 61.1), turned to 90 degrees
- moved IC5 24.5 mm to (128.4, 86.4), turned to 90 degrees
Connections:
- net /peripherals/CD_IN renamed /peripherals/CD_IN_RS232
- net /peripherals/SERIAL_DATA_IN renamed /peripherals/SERIAL_DATA_IN_RS232
- net /peripherals/SER_DATA_OUT renamed /peripherals/SERIAL_OUT_RS232
- net /video/S renamed Net-(C34-Pad2)
- CN2 pad 15: Net-(CN2-Pad15) -> /peripherals/K15
- IC4 pad 10: /gime/SERINT -> Net-(IC4-Pad10)
- IC4 pad 11: Net-(IC4-Pad11) -> /gime/SERINT
- IC4 pad 12: Net-(CN2-Pad15) -> Net-(IC4-Pad12)
- IC4 pad 13: /peripherals/RGB_OUT_10 -> /peripherals/K15
- IC4 pad 14: Net-(IC4-Pad14) -> /peripherals/RGB_OUT_10
- IC4 pad 18: /~CART -> Net-(IC4-Pad18)
- IC4 pad 19: Net-(IC4-Pad19) -> /~CART
- IC4 pad 2: /peripherals/CASS_DATA_OUT_TTL -> Net-(IC4-Pad2)
- IC4 pad 20: +5V -> Net-(IC4-Pad20)
- IC4 pad 21: /R~W -> +5V
- IC4 pad 22: /peripherals/HI -> Net-(IC4-Pad22)
- IC4 pad 23: /gime/PIA_~CS2 -> /R~W
- IC4 pad 24: /A5 -> /peripherals/HI
- IC4 pad 25: /ECLK -> /gime/PIA_~CS2
- IC4 pad 26: /D7 -> /A5
- IC4 pad 27: /D6 -> Net-(IC4-Pad27)
- IC4 pad 28: /D5 -> /ECLK
- IC4 pad 29: /D4 -> /D7
- IC4 pad 3: /peripherals/SER_DATA_IN_TTL -> /peripherals/CASS_DATA_IN_TTL
- IC4 pad 30: /D3 -> /D6
- IC4 pad 31: /D2 -> /D5
- IC4 pad 32: /D1 -> /D4
- IC4 pad 33: /D0 -> /D3
- IC4 pad 34: /~RESET -> /D2
- IC4 pad 35: /A1 -> /D1
- IC4 pad 36: /A0 -> /D0
- IC4 pad 37: /~FIRQ -> /~RESET
- IC4 pad 38: /~FIRQ -> /A1
- IC4 pad 39: /peripherals/CASS_M_IN_TTL -> /A0
- IC4 pad 4: Net-(IC4-Pad4) -> /peripherals/SER_OUT_TTL
- IC4 pad 40: /peripherals/CD_OUT_TTL -> Net-(IC4-Pad40)
- IC5 pad 10: Net-(CN2-Pad9) -> /peripherals/PA7
- IC5 pad 11: Net-(CN2-Pad10) -> Net-(CN2-Pad9)
- IC5 pad 12: Net-(CN2-Pad11) -> Net-(CN2-Pad10)
- IC5 pad 13: Net-(CN2-Pad12) -> Net-(CN2-Pad11)
- IC5 pad 14: Net-(CN2-Pad13) -> Net-(CN2-Pad12)
- IC5 pad 15: Net-(CN2-Pad14) -> Net-(CN2-Pad13)
- IC5 pad 16: Net-(CN2-Pad15) -> Net-(CN2-Pad14)
- IC5 pad 17: Net-(CN2-Pad16) -> /peripherals/K15
- IC5 pad 18: /gime/~VSYNC -> Net-(CN2-Pad16)
- IC5 pad 19: /peripherals/SELB -> /gime/~VSYNC
- IC5 pad 2: /peripherals/KR1 -> Net-(IC5-Pad2)
- IC5 pad 20: +5V -> /peripherals/SELB
- IC5 pad 21: /R~W -> +5V
- IC5 pad 22: /peripherals/HI -> Net-(IC5-Pad22)
- IC5 pad 23: /gime/PIA_~CS2 -> /R~W
- IC5 pad 24: Net-(IC15-Pad4) -> /peripherals/HI
- IC5 pad 25: /ECLK -> /gime/PIA_~CS2
- IC5 pad 26: /D7 -> Net-(IC15-Pad4)
- IC5 pad 27: /D6 -> Net-(IC5-Pad27)
- IC5 pad 28: /D5 -> /ECLK
- IC5 pad 29: /D4 -> /D7
- IC5 pad 3: /peripherals/KR2 -> /peripherals/KR1
- IC5 pad 30: /D3 -> /D6
- IC5 pad 31: /D2 -> /D5
- IC5 pad 32: /D1 -> /D4
- IC5 pad 33: /D0 -> /D3
- IC5 pad 34: /~RESET -> /D2
- IC5 pad 35: /A1 -> /D1
- IC5 pad 36: /A0 -> /D0
- IC5 pad 37: /~IRQ -> /~RESET
- IC5 pad 38: /~IRQ -> /A1
- IC5 pad 39: /peripherals/SELA -> /A0
- IC5 pad 4: /peripherals/KR3 -> /peripherals/KR2
- IC5 pad 40: /gime/~HSYNC -> Net-(IC5-Pad40)
- IC5 pad 5: /peripherals/KR4 -> /peripherals/KR3
- IC5 pad 6: /peripherals/KR5 -> /peripherals/KR4
- IC5 pad 7: /peripherals/KR6 -> /peripherals/KR5
- IC5 pad 8: /peripherals/KR7 -> /peripherals/KR6
- IC5 pad 9: /peripherals/PA7 -> /peripherals/KR7
- IC7 pad 2: Net-(IC4-Pad19) -> Net-(IC4-Pad20)
- IC7 pad 3: Net-(IC4-Pad4) -> Net-(IC4-Pad5)
- IC7 pad 4: Net-(IC4-Pad5) -> Net-(IC4-Pad6)
- IC7 pad 5: Net-(IC4-Pad6) -> Net-(IC4-Pad7)
- IC7 pad 6: Net-(IC4-Pad7) -> Net-(IC4-Pad8)
- IC7 pad 7: Net-(IC4-Pad8) -> Net-(IC4-Pad9)
- IC7 pad 8: Net-(IC4-Pad9) -> Net-(IC4-Pad10)
- IC8 pad 10: /peripherals/CASS_M_IN_TTL -> /peripherals/CASS_M_ON_TTL
- IC8 pad 5: /peripherals/CD_OUT_TTL -> /peripherals/CD_IN_TTL
- IC8 pad 6: /peripherals/SER_DATA_IN_TTL -> /peripherals/SER_OUT_TTL
- IC8 pad 7: /peripherals/CASS_DATA_OUT_TTL -> /peripherals/CASS_DATA_IN_TTL
- R12 pad 2: Net-(IC4-Pad11) -> Net-(IC4-Pad12)
- R59 pad 2: Net-(CN2-Pad15) -> /peripherals/K15
Routing:
- net GNDS: track 1598.2 -> 0.00 mm, vias 5 -> 0
- net +5V: track 955.2 -> 0.00 mm, vias 1 -> 0
- net /D5: track 453.9 -> 0.00 mm, vias 11 -> 0
- net /D4: track 411.8 -> 0.00 mm, vias 4 -> 0
- net /D3: track 396.0 -> 0.00 mm, vias 4 -> 0
- net /D2: track 380.1 -> 0.00 mm, vias 3 -> 0
- net /~CART: track 376.3 -> 0.00 mm, vias 12 -> 0
- net /D0: track 375.3 -> 0.00 mm, vias 4 -> 0
- net /D6: track 370.1 -> 0.00 mm, vias 5 -> 0
- net /D7: track 369.0 -> 0.00 mm, vias 3 -> 0
- net /D1: track 356.8 -> 0.00 mm, vias 4 -> 0
- net /A1: track 341.7 -> 0.00 mm, vias 5 -> 0
- net /~RESET: track 326.3 -> 0.00 mm, vias 3 -> 0
- net 8V: track 318.8 -> 0.00 mm, vias 3 -> 0
- net /ECLK: track 310.9 -> 0.00 mm, vias 5 -> 0
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- removed copper zone on B.Cu, net (none)
- removed copper zone on F.Cu, net GNDS

Commit message: -repplaced a whole bunch of THT components with SMT components
Parts:
- C1, C10, C11, C12, C13, C14, C18, C19, C22, C23, C26, C28, C30, C37, C38, C39, C4, C40, C41, C42, C47, C48, C50, C51, C58, C59, C6, C61, C68, C7, C8: footprint Capacitor_THT:C_Disc_D4.7mm_W2.5mm_P5.00mm -> Capacitor_SMD:C_0805_2012Metric_Pad1.18x1.45mm_HandSolder
- C15, C27: footprint Capacitor_THT:CP_Radial_D8.0mm_P5.00mm -> Capacitor_SMD:CP_Elec_6.3x5.3
- C16, C17, C20, C21, C25, C32, C33, C35, C36, C49: footprint Capacitor_THT:C_Disc_D8.0mm_W2.5mm_P5.00mm -> Capacitor_SMD:C_0805_2012Metric_Pad1.18x1.45mm_HandSolder
- C2, C55, C56: footprint Capacitor_THT:CP_Radial_D5.0mm_P2.00mm -> Capacitor_SMD:CP_Elec_4x5.3
- C29: value 4700uF 16V -> 4700uF 25V; footprint Capacitor_THT:CP_Radial_D12.5mm_P5.00mm -> Capacitor_SMD:CP_Elec_4x5.3
- C3: footprint Capacitor_THT:CP_Radial_D5.0mm_P2.00mm -> Capacitor_SMD:CP_Elec_4x5.4
- C31: value 220uF 16V -> 220uF 25V; footprint Capacitor_THT:CP_Radial_D8.0mm_P5.00mm -> Capacitor_SMD:CP_Elec_8x10
- C34: footprint Capacitor_THT:C_Disc_D4.3mm_W1.9mm_P5.00mm -> Capacitor_SMD:C_0805_2012Metric_Pad1.18x1.45mm_HandSolder
- C5, C52, C53, C57: footprint Capacitor_THT:C_Axial_L5.1mm_D3.1mm_P10.00mm_Horizontal -> Capacitor_SMD:C_0805_2012Metric_Pad1.18x1.45mm_HandSolder
- C54: value 470uF -> 470uF 16V; footprint Capacitor_THT:CP_Radial_D8.0mm_P3.50mm -> Capacitor_SMD:CP_Elec_8x10
- C60: footprint Capacitor_THT:C_Rect_L7.2mm_W3.0mm_P5.00mm_FKS2_FKP2_MKS2_MKP2 -> Capacitor_SMD:C_0805_2012Metric_Pad1.18x1.45mm_HandSolder
- C62, C63: footprint Capacitor_THT:CP_Radial_D8.0mm_P3.50mm -> Capacitor_SMD:CP_Elec_8x10
- C64: footprint Capacitor_THT:C_Rect_L7.2mm_W2.5mm_P5.00mm_FKS2_FKP2_MKS2_MKP2 -> Capacitor_SMD:C_0805_2012Metric_Pad1.18x1.45mm_HandSolder
- C9: footprint Capacitor_THT:CP_Radial_D5.0mm_P2.00mm -> Capacitor_SMD:CP_Elec_6.3x5.3
- IC10, IC11, IC12, IC13, IC3: footprint Package_DIP:DIP-20_W7.62mm_Socket -> Package_SO:SOIC-20W_7.5x12.8mm_P1.27mm
- IC14, IC15: footprint Package_DIP:DIP-14_W7.62mm_Socket -> Package_SO:SOIC-14_3.9x8.7mm_P1.27mm
- IC9: footprint Package_DIP:DIP-16_W7.62mm_Socket -> Package_SO:SOP-16_3.9x9.9mm_P1.27mm
- R11, R16, R17, R2, R21, R22, R24, R28, R3, R30, R33, R34, R35, R36, R38, R39, R4, R40, R42, R43, R45, R46, R47, R49, R5, R50, R52, R53, R54, R56, R57, R59, R6, R61, R62, R68, R69, R7, R71, R72, R8: footprint Resistor_THT:R_Axial_DIN0207_L6.3mm_D2.5mm_P10.16mm_Horizontal -> Resistor_SMD:R_1206_3216Metric_Pad1.30x1.75mm_HandSolder
- R15: footprint Resistor_THT:R_Axial_DIN0204_L3.6mm_D1.6mm_P7.62mm_Horizontal -> Resistor_SMD:R_2010_5025Metric_Pad1.40x2.65mm_HandSolder
- moved IC4 80.9 mm to (126.2, 142.0)
- moved C39 38.8 mm to (144.2, 53.1)
- moved C41 38.5 mm to (143.8, 70.0)
- moved IC10 32.9 mm to (152.4, 89.3)
- moved IC5 30.4 mm to (126.2, 116.7)
- moved IC11 25.5 mm to (132.7, 53.5)
- moved IC13 24.4 mm to (132.5, 70.9)
- moved IC12 23.8 mm to (132.0, 88.6)
- moved C40 18.7 mm to (163.5, 89.5)
- moved IC3 8.56 mm to (284.1, 66.6)
- moved IC9 6.06 mm to (244.1, 136.4)
- moved IC15 5.09 mm to (167.0, 153.8)
- moved IC14 4.61 mm to (166.5, 141.2)
- moved C14 4.47 mm to (46.6, 159.2)
- moved C15 3.85 mm to (55.1, 162.2)
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
Commit message: -converted more components from THT to SMD -replaced SALT chip with replacement circuitry
Parts:
- removed C30: .1uF, Capacitor_SMD:C_0805_2012Metric_Pad1.18x1.45mm_HandSolder
- removed C31, C62: 220uF 25V, Capacitor_SMD:CP_Elec_8x10
- removed C32, C33, C35: .022uF, Capacitor_SMD:C_0805_2012Metric_Pad1.18x1.45mm_HandSolder
- removed D1, D2: 1N5401-G, Diode_THT:D_DO-201AD_P15.24mm_Horizontal
- removed D13, D14: 1N4002, Diode_THT:D_DO-41_SOD81_P10.16mm_Horizontal
- removed D3, D4: UF1002-T, Diode_THT:D_DO-41_SOD81_P10.16mm_Horizontal
- removed D6, D7: 1N5228B-TAP, Diode_THT:D_DO-35_SOD27_P7.62mm_Horizontal
- removed FB1, FB2, FB7: , coco2:FB_28L0138-10R-10
- removed IC8: SC77527P, Package_DIP:DIP-16_W7.62mm_Socket
- removed J5A1001: CVIDEO, coco2:KLPX-0848A-2-R
- removed J5B1001: SOUND, coco2:KLPX-0848A-2-R
- removed Q1: 2N6123, Package_TO_SOT_THT:TO-220-3_Horizontal_TabDown
- removed R15: 270 1/2W, Resistor_SMD:R_2010_5025Metric_Pad1.40x2.65mm_HandSolder
- removed R16, R17: 1K, Resistor_SMD:R_1206_3216Metric_Pad1.30x1.75mm_HandSolder
- removed R18: 510, Resistor_THT:R_Axial_DIN0207_L6.3mm_D2.5mm_P10.16mm_Horizontal
- removed R19: .1 ohms 1/2W, Resistor_THT:R_Axial_DIN0411_L9.9mm_D3.6mm_P15.24mm_Horizontal
- removed R20: 51, Resistor_THT:R_Axial_DIN0207_L6.3mm_D2.5mm_P10.16mm_Horizontal
- removed TP1: 5V, TestPoint:TestPoint_Pad_3.0x3.0mm
- added C1001: .1uF, Capacitor_SMD:C_0805_2012Metric_Pad1.18x1.45mm_HandSolder, F.Cu at (154.5, 66.3)
- added C1002: .47uF, Capacitor_SMD:C_0805_2012Metric_Pad1.18x1.45mm_HandSolder, F.Cu at (155.1, 71.1)
- added C1003: .47uF, Capacitor_SMD:C_0805_2012Metric_Pad1.18x1.45mm_HandSolder, F.Cu at (161.6, 63.1)
- added C1004: .47uF, Capacitor_SMD:C_0805_2012Metric_Pad1.18x1.45mm_HandSolder, F.Cu at (152.2, 75.1)
- added D1001: 5A 40V, Diode_SMD:D_SMB, F.Cu at (74.9, 151.7)
- added D1002: 1N4148, Diode_SMD:D_SOD-323F, F.Cu at (58.3, 128.8)
- added J5: SJ-435107RS, coco2:CUI_SJ-435107RS, F.Cu at (218.3, 22.6)
- added L1001: 33uH, Inductor_SMD:L_Sumida_CDMC6D28_7.25x6.5mm, F.Cu at (67.9, 151.1)
- added Q1001: MMBT9014C, Package_TO_SOT_SMD:SOT-23, F.Cu at (190.9, 60.8)
- added R1001: 10k, Resistor_SMD:R_1206_3216Metric_Pad1.30x1.75mm_HandSolder, F.Cu at (191.0, 65.0)
- added R1002: 100K, Resistor_SMD:R_1206_3216Metric_Pad1.30x1.75mm_HandSolder, F.Cu at (48.4, 107.0)
- added R1003: 100K, Resistor_SMD:R_1206_3216Metric_Pad1.30x1.75mm_HandSolder, F.Cu at (57.1, 102.5)
- added R1004: 5.1K, Resistor_SMD:R_1206_3216Metric_Pad1.30x1.75mm_HandSolder, F.Cu at (65.9, 97.9)
- added R1005: 5.1K, Resistor_SMD:R_1206_3216Metric_Pad1.30x1.75mm_HandSolder, F.Cu at (64.5, 128.9)
- added R1006: 5.1K, Resistor_SMD:R_1206_3216Metric_Pad1.30x1.75mm_HandSolder, F.Cu at (63.1, 102.5)
- added R1007: 20M, Resistor_SMD:R_1206_3216Metric_Pad1.30x1.75mm_HandSolder, F.Cu at (57.5, 114.3)
- added R1008: 10k, Resistor_SMD:R_1206_3216Metric_Pad1.30x1.75mm_HandSolder, F.Cu at (53.3, 119.9)
- added TP1001: 5V, TestPoint:TestPoint_Pad_3.0x3.0mm, F.Cu at (38.8, 76.7)
- added U1001: LM2596S-5, Package_TO_SOT_SMD:TO-263-5_TabPin3, F.Cu at (52.2, 153.0)
- added U1002: MAX3232, Package_SO:SOIC-16_3.9x9.9mm_P1.27mm, F.Cu at (161.6, 71.1)
- added U1003: LM393, Package_SO:TSSOP-8_4.4x3mm_P0.65mm, F.Cu at (67.8, 119.3)
- C15: value 100uF 16v -> 220uF 25V; footprint Capacitor_SMD:CP_Elec_6.3x5.3 -> Capacitor_SMD:CP_Elec_8x10
- C29: footprint Capacitor_SMD:CP_Elec_4x5.3 -> Capacitor_SMD:CP_Elec_18x22
- CN7: value Conn_01x03_Male -> Jack-DC; footprint Connector_Molex:Molex_KK-396_A-41791-0003_1x03_P3.96mm_Vertical -> Connector_BarrelJack:BarrelJack_CUI_PJ-063AH_Horizontal
- D12, D5: footprint Diode_THT:D_DO-35_SOD27_P7.62mm_Horizontal -> Diode_SMD:D_SOD-323F
- R1, R12, R23, R27, R29, R31, R32, R64, R65, R66, R70: footprint Resistor_THT:R_Axial_DIN0207_L6.3mm_D2.5mm_P10.16mm_Horizontal -> Resistor_SMD:R_1206_3216Metric_Pad1.30x1.75mm_HandSolder
- R10, R63, R9: footprint Resistor_THT:R_Axial_DIN0309_L9.0mm_D3.2mm_P12.70mm_Horizontal -> Resistor_SMD:R_1206_3216Metric_Pad1.30x1.75mm_HandSolder
- R13: value 100 1/2W -> 100 1W; footprint Resistor_THT:R_Axial_DIN0411_L9.9mm_D3.6mm_P12.70mm_Horizontal -> Resistor_SMD:R_2512_6332Metric_Pad1.40x3.35mm_HandSolder
- R14: value 220 1/2W -> 220 1W; footprint Resistor_THT:R_Axial_DIN0411_L9.9mm_D3.6mm_P12.70mm_Horizontal -> Resistor_SMD:R_2512_6332Metric_Pad1.40x3.35mm_HandSolder
- moved CN7 196.8 mm to (279.9, 17.9), turned to 0 degrees
- moved R66 125.3 mm to (160.4, 78.7), turned to 0 degrees
- moved C14 76.4 mm to (18.7, 88.0), turned to 0 degrees
- moved SW2 47.7 mm to (235.8, 21.8)
- moved C13 47.7 mm to (115.3, 184.6)
- moved R24 47.7 mm to (108.5, 177.1)
- moved C29 39.5 mm to (87.7, 148.6), turned to 90 degrees
- moved R7 35.4 mm to (75.6, 189.1)
- moved R12 35.4 mm to (75.6, 186.0)
- moved C54 33.4 mm to (201.4, 28.1), turned to 90 degrees
- moved D5 28.0 mm to (196.4, 50.1), turned to 270 degrees
- moved C28 25.0 mm to (65.1, 161.1), turned to 270 degrees
- moved C15 24.0 mm to (68.4, 142.2), turned to 0 degrees
- moved C36 14.5 mm to (102.4, 80.2)
- moved Q2 11.9 mm to (234.4, 47.0)
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Connections:
- C28 pad 1: /peripherals/+SALT_VIN -> /power/12VDC
- C29 pad 1: /peripherals/+SALT_VIN -> /power/12VDC
- C36 pad 1: Net-(C36-Pad1) -> GNDS
- C54 pad 2: Net-(C54-Pad2) -> /video/CVIDEO_OUT
- C63 pad 1: Net-(C63-Pad1) -> /power/12VDC
- CN7 pad 1: Net-(CN7-Pad1) -> /power/12VDC_PS
- CN7 pad 2: GNDS -> /power/GND_PS
- IC36 pad 3: Net-(C63-Pad1) -> /power/12VDC
- JK3 pad 1: Net-(JK3-Pad1) -> /peripherals/CD_IN_RS232
- JK3 pad 2: Net-(JK3-Pad2) -> /peripherals/SERIAL_DATA_IN_RS232
- JK3 pad 4: Net-(FB7-Pad2) -> /peripherals/SERIAL_OUT_RS232
- SW1 pad 2: Net-(C36-Pad1) -> /power/GND_PS
- SW1 pad 3: Net-(CN7-Pad3) -> GNDS
- SW1 pad 5: Net-(C35-Pad1) -> /power/12VDC_PS
- SW1 pad 6: Net-(CN7-Pad1) -> /power/12VDC
Routing:
- net /power/12VDC_PS: track 0.00 -> 195.8 mm
- net /power/12VDC: track 0.00 -> 155.2 mm
- net Net-(D1001-Pad1): track 0.00 -> 23.4 mm
- net GNDS: track 0.00 -> 19.7 mm
- net +5V: track 0.00 -> 17.8 mm

Commit message: routed the board
Parts:
- removed CN4, CN5, CN6: Conn_01x12_Female, coco2:PinSocket_1x12_P2.54mm_for_memory_board_adapter
- added BREAKOUT0: Conn_01x18_Male, Connector_PinHeader_2.54mm:PinHeader_1x18_P2.54mm_Vertical, F.Cu at (154.4, 117.1)
- added CN4000: Conn_01x12_Female, Connector_PinSocket_2.54mm:PinSocket_1x12_P2.54mm_Vertical, F.Cu at (157.6, 108.1)
- added CN56: Conn_01x24_Female, Connector_PinSocket_2.54mm:PinSocket_1x24_P2.54mm_Vertical, F.Cu at (116.8, 102.6)
- added D1003: 1N4148, Diode_SMD:D_SOD-323F, F.Cu at (250.3, 36.4)
- added D1004: 1N4148, Diode_SMD:D_SOD-323F, F.Cu at (244.9, 36.4)
- added J1001: RGB_2_ADAPTER_ADAPTER, Connector_PinHeader_2.54mm:PinHeader_2x03_P2.54mm_Horizontal, F.Cu at (254.3, 29.5)
- added J1002: Conn_01x04_Male, Connector_PinHeader_2.54mm:PinHeader_1x04_P2.54mm_Vertical, F.Cu at (176.4, 84.4)
- C2, C55, C56: value 10uF 25v -> 10uF 16v; footprint Capacitor_SMD:CP_Elec_4x5.3 -> Capacitor_Tantalum_SMD:CP_EIA-3216-18_Kemet-A
- C27: value 100uF 16v -> 100uF 6.3V; footprint Capacitor_SMD:CP_Elec_6.3x5.3 -> Capacitor_Tantalum_SMD:CP_EIA-3528-21_Kemet-B
- C3: value 1uF 50V -> 10uF 16v; footprint Capacitor_SMD:CP_Elec_4x5.4 -> Capacitor_Tantalum_SMD:CP_EIA-3216-18_Kemet-A
- R1004, R1005, R1006: footprint Resistor_SMD:R_1206_3216Metric_Pad1.30x1.75mm_HandSolder -> Resistor_SMD:R_0805_2012Metric_Pad1.20x1.40mm_HandSolder
- moved TP1001 218.6 mm to (255.5, 105.2)
- moved C13 76.2 mm to (108.7, 108.6)
- moved R7 73.5 mm to (143.1, 159.9)
- moved R24 68.6 mm to (115.3, 108.8)
- moved C14 65.7 mm to (76.5, 119.3), turned to 90 degrees
- moved C38 64.0 mm to (147.1, 88.6)
- moved R12 58.5 mm to (115.4, 143.1)
- moved C40 40.1 mm to (123.4, 88.6)
- moved R6 34.5 mm to (152.7, 131.6)
- moved R1002 26.1 mm to (64.1, 127.9), turned to 90 degrees
- moved R1006 25.8 mm to (58.7, 127.9), turned to 270 degrees
- moved MP1 22.8 mm to (296.8, 73.5), turned to 270 degrees
- moved C39 20.8 mm to (123.4, 53.5)
- moved MP2 20.4 mm to (293.3, 73.5), turned to 270 degrees
- moved C41 20.4 mm to (123.4, 71.0)
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Connections:
- CN7 pad 2: /power/GND_PS -> GNDS
- IC1 pad 6: Net-(IC1-Pad6) -> /cpu/BUS_TXRX_ENABLE
- IC3 pad 19: GNDS -> /cpu/BUS_TXRX_ENABLE
- IC4 pad 15: Net-(IC4-Pad15) -> /peripherals/IC4_PB4
- IC4 pad 16: Net-(IC4-Pad16) -> /peripherals/IC4_PB5
- IC4 pad 17: Net-(IC4-Pad17) -> /peripherals/IC4_PB6
- IC4 pad 18: Net-(IC4-Pad18) -> /peripherals/IC4_PB7
- SW1 pad 2: /power/GND_PS -> GNDS
Routing:
- net GNDS: track 19.7 -> 1528.3 mm, vias 0 -> 85
- net +5V: track 17.8 -> 1034.7 mm, vias 0 -> 56
- net /D4: track 0.00 -> 484.8 mm, vias 0 -> 10
- net /D2: track 0.00 -> 456.0 mm, vias 0 -> 8
- net /D6: track 0.00 -> 452.8 mm, vias 0 -> 11
- net /D0: track 0.00 -> 450.0 mm, vias 0 -> 10
- net /D5: track 0.00 -> 421.1 mm, vias 0 -> 10
- net /D1: track 0.00 -> 420.7 mm, vias 0 -> 12
- net /D3: track 0.00 -> 391.4 mm, vias 0 -> 12
- net /~RESET: track 0.00 -> 389.5 mm, vias 0 -> 6
- net /D7: track 0.00 -> 385.1 mm, vias 0 -> 10
- net /A1: track 0.00 -> 375.4 mm, vias 0 -> 5
- net /R~W: track 0.00 -> 357.9 mm, vias 0 -> 4
- net /ECLK: track 0.00 -> 331.7 mm, vias 0 -> 8
- net /A0: track 0.00 -> 309.2 mm, vias 0 -> 1
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- added copper zone on B.Cu, net GNDS
- added copper zone on F.Cu, net GNDS
Other:
- board text added: "+5V"
- board text added: "FROM IC4"
- board text added: "PA0"
- board text added: "PA1"
- board text added: "PA2"
- board text added: "PA3"
- board text added: "PA4"
- board text added: "PA5"
- board text added: "PA6"
- board text added: "PB0"
- board text added: "PB1"
- board text added: "PB2"
- board text added: "PB3"
- board text added: "PB4"
- board text added: "PB5"
- board text added: "PB6"
- board text added: "PB7"
