File: coco3/coco3.kicad_pcb (KiCad board)
At the start: 2 copper layers, 280 x 155.3 mm, 196 parts, among them CN1 Conn_02x20_Odd_Even, CN2 Conn_01x16_Female, CN3 Conn_02x05_Odd_Even, CN4000 Conn_01x12_Female, CN56 Conn_01x24_Female, CN7 Jack-DC, IC1 MC6809E, IC10 74LS244, IC11 74LS244, IC12 74LS244, IC13 74LS374, IC14 74LS30, IC15 74LS04, IC2 27C256, IC3 SN74LS245N, IC36 MC78L08_TO92, IC4 W65C21N6TPLG-14, IC5 W65C21N6TPLG-14, IC6 TCC1014, IC7 SC77526, IC9 74LS138, J1001 RGB_2_ADAPTER_ADAPTER, J1002 Conn_01x04_Male, J5 SJ-435107RS, Q1001 MMBT9014C, Q2 2SC945(NTE85), Q3 2SC945(NTE85), Q4 MPSA13(NTE46), Q5 2SC945(NTE85), Q6 2SC945(NTE85), Q7 2SC945(NTE85), SW1 SW_DPDT_x2, SW2 Reset Switch, U1001 LM2596S-5, U1002 MAX3232, U1003 LM393, X1 28.63636 MHz

Commit message: added replacement circuitry for SC77526P DAC/ADC chip
Parts:
- removed IC7: SC77526, Package_DIP:DIP-20_W7.62mm_Socket
- removed U1003: LM393, Package_SO:TSSOP-8_4.4x3mm_P0.65mm
- added C30: 20pF, Capacitor_SMD:C_0805_2012Metric_Pad1.18x1.45mm_HandSolder, F.Cu at (91.1, 122.5)
- added R15: 100K, Resistor_SMD:R_0603_1608Metric_Pad0.98x0.95mm_HandSolder, F.Cu at (83.9, 122.8)
- added R16: 330K, Resistor_SMD:R_0805_2012Metric_Pad1.20x1.40mm_HandSolder, F.Cu at (96.7, 125.9)
- added R17: 160K, Resistor_SMD:R_0603_1608Metric_Pad0.98x0.95mm_HandSolder, F.Cu at (96.7, 130.4)
- added R18: 82K, Resistor_SMD:R_0805_2012Metric_Pad1.20x1.40mm_HandSolder, F.Cu at (93.2, 119.9)
- added R19: 82K, Resistor_SMD:R_0805_2012Metric_Pad1.20x1.40mm_HandSolder, F.Cu at (96.7, 134.9)
- added R20: 40.2K, Resistor_SMD:R_0603_1608Metric_Pad0.98x0.95mm_HandSolder, F.Cu at (116.2, 135.3)
- added R25: 300K, Resistor_SMD:R_0805_2012Metric_Pad1.20x1.40mm_HandSolder, F.Cu at (100.4, 120.3)
- added R26: 20K, Resistor_SMD:R_0805_2012Metric_Pad1.20x1.40mm_HandSolder, F.Cu at (116.2, 130.1)
- added R37: 10K, Resistor_SMD:R_0805_2012Metric_Pad1.20x1.40mm_HandSolder, F.Cu at (116.2, 125.4)
- added R41: 10K, Resistor_SMD:R_0805_2012Metric_Pad1.20x1.40mm_HandSolder, F.Cu at (78.7, 109.0)
- added R44: 10M, Resistor_SMD:R_0805_2012Metric_Pad1.20x1.40mm_HandSolder, F.Cu at (58.4, 119.4)
- added R48: 1K, Resistor_SMD:R_0805_2012Metric_Pad1.20x1.40mm_HandSolder, F.Cu at (63.5, 115.0)
- added U1: 74LS367, Package_SO:SOIC-16_3.9x9.9mm_P1.27mm, F.Cu at (108.2, 130.8)
- added U2: TS5A3166DBVR, Package_TO_SOT_SMD:SOT-23-5, F.Cu at (102.9, 117.0)
- added U3: LM393, Package_SO:TSSOP-8_4.4x3mm_P0.65mm, F.Cu at (65.1, 119.9)
- added U4: CD4052B, Package_SO:HTSSOP-16-1EP_4.4x5mm_P0.65mm_EP3x3mm, F.Cu at (90.4, 113.8)
Connections:
- C24 pad 2: Net-(C24-Pad2) -> /peripherals/Color Computer DAC/CASSETTE_SND_IN
- CN1 pad 1: Net-(CN1-Pad1) -> (no net)
- CN1 pad 2: Net-(CN1-Pad2) -> (no net)
- CN3 pad 6: Net-(CN3-Pad6) -> (no net)
- FB6 pad 1: Net-(FB6-Pad1) -> /peripherals/Color Computer DAC/CASSETTE_OUT
- IC1 pad 33: Net-(IC1-Pad33) -> (no net)
- IC1 pad 36: Net-(IC1-Pad36) -> (no net)
- IC1 pad 38: Net-(IC1-Pad38) -> (no net)
- IC1 pad 5: Net-(IC1-Pad5) -> (no net)
- IC2 pad 1: Net-(IC2-Pad1) -> (no net)
- IC4 pad 10: Net-(IC4-Pad10) -> /peripherals/Color Computer DAC/D5
- IC4 pad 2: Net-(IC4-Pad2) -> (no net)
- IC4 pad 20: Net-(IC4-Pad20) -> /peripherals/Color Computer DAC/SND_ENABLE
- IC4 pad 22: Net-(IC4-Pad22) -> (no net)
- IC4 pad 27: Net-(IC4-Pad27) -> (no net)
- IC4 pad 40: Net-(IC4-Pad40) -> (no net)
- IC4 pad 5: Net-(IC4-Pad5) -> /peripherals/Color Computer DAC/D0
- IC4 pad 6: Net-(IC4-Pad6) -> /peripherals/Color Computer DAC/D1
- IC4 pad 7: Net-(IC4-Pad7) -> /peripherals/Color Computer DAC/D2
- IC4 pad 8: Net-(IC4-Pad8) -> /peripherals/Color Computer DAC/D3
- IC4 pad 9: Net-(IC4-Pad9) -> /peripherals/Color Computer DAC/D4
- IC5 pad 2: Net-(IC5-Pad2) -> (no net)
- IC5 pad 22: Net-(IC5-Pad22) -> (no net)
- IC5 pad 27: Net-(IC5-Pad27) -> (no net)
- IC5 pad 40: Net-(IC5-Pad40) -> (no net)
- IC9 pad 10: Net-(IC9-Pad10) -> (no net)
- IC9 pad 11: Net-(IC9-Pad11) -> (no net)
- IC9 pad 12: Net-(IC9-Pad12) -> (no net)
- IC9 pad 7: Net-(IC9-Pad7) -> (no net)
- J5 pad 5: Net-(J5-Pad5) -> (no net)
- J5 pad 6: Net-(J5-Pad6) -> (no net)
- RY1 pad 12: Net-(RY1-Pad12) -> (no net)
- SW1 pad 1: Net-(SW1-Pad1) -> (no net)
- SW1 pad 4: Net-(SW1-Pad4) -> (no net)
- U1002 pad 11: Net-(U1002-Pad11) -> (no net)
- U1002 pad 14: Net-(U1002-Pad14) -> (no net)
Routing:
- net GNDS: track 1528.3 -> 0.00 mm, vias 85 -> 0
- net +5V: track 1034.7 -> 0.00 mm, vias 56 -> 0
- net /D4: track 484.8 -> 0.00 mm, vias 10 -> 0
- net /D2: track 456.0 -> 0.00 mm, vias 8 -> 0
- net /D6: track 452.8 -> 0.00 mm, vias 11 -> 0
- net /D0: track 450.0 -> 0.00 mm, vias 10 -> 0
- net /D5: track 421.1 -> 0.00 mm, vias 10 -> 0
- net /D1: track 420.7 -> 0.00 mm, vias 12 -> 0
- net /D3: track 391.4 -> 0.00 mm, vias 12 -> 0
- net /~RESET: track 389.5 -> 0.00 mm, vias 6 -> 0
- net /D7: track 385.1 -> 0.00 mm, vias 10 -> 0
- net /A1: track 375.4 -> 0.00 mm, vias 5 -> 0
- net /R~W: track 357.9 -> 0.00 mm, vias 4 -> 0
- net /ECLK: track 331.7 -> 0.00 mm, vias 8 -> 0
- net /A0: track 309.2 -> 0.00 mm, vias 1 -> 0
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