File: coco3/cpu.sch (KiCad schematic (older format))
At the start: 15 parts, among them IC1 MC6809E, IC3 SN74LS245N, SW2 Reset Switch

Commit message: -repplaced a whole bunch of THT components with SMT components
Parts:
- C1: footprint Capacitor_THT:C_Disc_D4.7mm_W2.5mm_P5.00mm -> Capacitor_SMD:C_0805_2012Metric_Pad1.18x1.45mm_HandSolder; Manufacturer part# FG28C0G1H103JNT06 -> CL21A106KAYNNNE; Vendor digikey -> JLCPCB; Vendor part# 445-173474-1-ND -> C15850
- C2: footprint Capacitor_THT:CP_Radial_D5.0mm_P2.00mm -> Capacitor_SMD:CP_Elec_4x5.3; Manufacturer part# UPW1E100MDD -> VE-100M1ETR-0405; Vendor digikey -> JLCPCB; Vendor part# 493-1809-ND -> C134721
- C3: footprint Capacitor_THT:CP_Radial_D5.0mm_P2.00mm -> Capacitor_SMD:CP_Elec_4x5.4; Manufacturer part# 515D105M050JA6AE3 -> RVT1H1R0M0405; Vendor digikey -> JLCPCB; Vendor part# 718-2229-ND -> C3348
- C5: footprint Capacitor_THT:C_Axial_L5.1mm_D3.1mm_P10.00mm_Horizontal -> Capacitor_SMD:C_0805_2012Metric_Pad1.18x1.45mm_HandSolder; Manufacturer part# C410C333K5R5TA7200 -> 0805B333K500NT; Vendor digikey -> JLCPCB; Vendor part# 399-4470-1-ND -> C1739
- IC1: Datasheet http://www.on-shore.com/wp-content/uploads/2015/09/ipg2.pdf -> (none); Manufacturer part# ED40DT -> Z-ICS0S40P-W000; Vendor digikey -> JLCPCB; Vendor part# ED3048-5-ND -> C132506
- IC3: footprint Package_DIP:DIP-20_W7.62mm_Socket -> Package_SO:SOIC-20W_7.5x12.8mm_P1.27mm; Manufacturer part# SN74LS245N -> SN74LS245DWR; Vendor digikey -> JLCPCB; Vendor part# 296-1655-5-ND -> C129580
- R2, R3, R4, R5: footprint Resistor_THT:R_Axial_DIN0207_L6.3mm_D2.5mm_P10.16mm_Horizontal -> Resistor_SMD:R_1206_3216Metric_Pad1.30x1.75mm_HandSolder; Manufacturer part# Stackpole Electronics Inc -> 1206W4F4701T5E; Vendor digikey -> JLCPCB; Vendor part# CF14JT4K70CT-ND -> C17936
Changed lines of the file:
@@
 F 1 "MC6809E" H 5550 6950 50  0000 C CNN
 F 2 "Package_DIP:DIP-40_W15.24mm_Socket" H 5300 4050 50  0001 C CNN
-F 3 "http://www.on-shore.com/wp-content/uploads/2015/09/ipg2.pdf" H 5200 6975 50  0001 C CNN
-F 4 "http://www.on-shore.com/wp-content/uploads/2015/09/ipg2.pdf" H 5300 5550 50  0001 C CNN "Datasheet"
-F 5 "digikey" H 5300 5550 50  0001 C CNN "Vendor"
-F 6 "ED3048-5-ND" H 5300 5550 50  0001 C CNN "Vendor part#"
-F 7 "ED40DT" H 5300 5550 50  0001 C CNN "Manufacturer part#"
+F 3 "https://datasheet.lcsc.com/lcsc/1810201609_Ckmtw-Shenzhen-Cankemeng-Z-ICS0S40P-W000_C132506.pdf" H 5200 6975 50  0001 C CNN
+F 4 "JLCPCB" H 5300 5550 50  0001 C CNN "Vendor"
+F 5 "C132506" H 5300 5550 50  0001 C CNN "Vendor part#"
+F 6 "Z-ICS0S40P-W000" H 5300 5550 50  0001 C CNN "Manufacturer part#"
 	1    5300 5550
 	1    0    0    -1
@@
 F 0 "C1" V 5671 4000 50  0000 C CNN
 F 1 ".1uF" V 5762 4000 50  0000 C CNN
-F 2 "Capacitor_THT:C_Disc_D4.7mm_W2.5mm_P5.00mm" H 5900 4000 50  0001 C CNN
-F 3 " https://product.tdk.com/info/en/catalog/datasheets/leadmlcc_halogenfree_fg_en.pdf?ref_disty=digikey" H 5900 4000 50  0001 C CNN
-F 4 "digikey" V 5900 4000 50  0001 C CNN "Vendor"
-F 5 "445-173474-1-ND" V 5900 4000 50  0001 C CNN "Vendor part#"
-F 6 "FG28C0G1H103JNT06" V 5900 4000 50  0001 C CNN "Manufacturer part#"
+F 2 "Capacitor_SMD:C_0805_2012Metric_Pad1.18x1.45mm_HandSolder" H 5900 4000 50  0001 C CNN
+F 3 "https://datasheet.lcsc.com/lcsc/1811121310_Samsung-Electro-Mechanics-CL21A106KAYNNNE_C15850.pdf" H 5900 4000 50  0001 C CNN
+F 4 "JLCPCB" V 5900 4000 50  0001 C CNN "Vendor"
+F 5 "C15850" V 5900 4000 50  0001 C CNN "Vendor part#"
+F 6 "CL21A106KAYNNNE" V 5900 4000 50  0001 C CNN "Manufacturer part#"
 	1    5900 4000
 	0    1    1    0
@@
 F 0 "R4" H 3168 5146 50  0000 L CNN
 F 1 "4.7K" H 3168 5055 50  0000 L CNN
-F 2 "Resistor_THT:R_Axial_DIN0207_L6.3mm_D2.5mm_P10.16mm_Horizontal" H 3100 5100 50  0001 C CNN
-F 3 "https://www.seielect.com/catalog/sei-cf_cfm.pdf" H 3100 5100 50  0001 C CNN
-F 4 "digikey" H 3100 5100 50  0001 C CNN "Vendor"
-F 5 "CF14JT4K70CT-ND  " H 3100 5100 50  0001 C CNN "Vendor part#"
-F 6 "Stackpole Electronics Inc" H 3100 5100 50  0001 C CNN "Manufacturer part#"
+F 2 "Resistor_SMD:R_1206_3216Metric_Pad1.30x1.75mm_HandSolder" H 3100 5100 50  0001 C CNN
+F 3 "https://datasheet.lcsc.com/lcsc/1810301414_UNI-ROYAL-Uniroyal-Elec-1206W4F4701T5E_C17936.pdf" H 3100 5100 50  0001 C CNN
+F 4 "JLCPCB" H 3100 5100 50  0001 C CNN "Vendor"
+F 5 "C17936" H 3100 5100 50  0001 C CNN "Vendor part#"
+F 6 "1206W4F4701T5E" H 3100 5100 50  0001 C CNN "Manufacturer part#"
 	1    3100 5100
 	1    0    0    -1
@@
 F 0 "R2" H 2868 5146 50  0000 L CNN
 F 1 "4.7K" H 2868 5055 50  0000 L CNN
-F 2 "Resistor_THT:R_Axial_DIN0207_L6.3mm_D2.5mm_P10.16mm_Horizontal" H 2800 5100 50  0001 C CNN
-F 3 "https://www.seielect.com/catalog/sei-cf_cfm.pdf" H 2800 5100 50  0001 C CNN
-F 4 "digikey" H 2800 5100 50  0001 C CNN "Vendor"
-F 5 "CF14JT4K70CT-ND  " H 2800 5100 50  0001 C CNN "Vendor part#"
-F 6 "Stackpole Electronics Inc" H 2800 5100 50  0001 C CNN "Manufacturer part#"
+F 2 "Resistor_SMD:R_1206_3216Metric_Pad1.30x1.75mm_HandSolder" H 2800 5100 50  0001 C CNN
+F 3 "https://datasheet.lcsc.com/lcsc/1810301414_UNI-ROYAL-Uniroyal-Elec-1206W4F4701T5E_C17936.pdf" H 2800 5100 50  0001 C CNN
+F 4 "JLCPCB" H 2800 5100 50  0001 C CNN "Vendor"
+F 5 "C17936" H 2800 5100 50  0001 C CNN "Vendor part#"
+F 6 "1206W4F4701T5E" H 2800 5100 50  0001 C CNN "Manufacturer part#"
 	1    2800 5100
 	1    0    0    -1
@@
 F 0 "R3" H 2568 5146 50  0000 L CNN
 F 1 "4.7K" H 2568 5055 50  0000 L CNN
-F 2 "Resistor_THT:R_Axial_DIN0207_L6.3mm_D2.5mm_P10.16mm_Horizontal" H 2500 5100 50  0001 C CNN
-F 3 "https://www.seielect.com/catalog/sei-cf_cfm.pdf" H 2500 5100 50  0001 C CNN
-F 4 "digikey" H 2500 5100 50  0001 C CNN "Vendor"
-F 5 "CF14JT4K70CT-ND  " H 2500 5100 50  0001 C CNN "Vendor part#"
-F 6 "Stackpole Electronics Inc" H 2500 5100 50  0001 C CNN "Manufacturer part#"
+F 2 "Resistor_SMD:R_1206_3216Metric_Pad1.30x1.75mm_HandSolder" H 2500 5100 50  0001 C CNN
+F 3 "https://datasheet.lcsc.com/lcsc/1810301414_UNI-ROYAL-Uniroyal-Elec-1206W4F4701T5E_C17936.pdf" H 2500 5100 50  0001 C CNN
+F 4 "JLCPCB" H 2500 5100 50  0001 C CNN "Vendor"
+F 5 "C17936" H 2500 5100 50  0001 C CNN "Vendor part#"
+F 6 "1206W4F4701T5E" H 2500 5100 50  0001 C CNN "Manufacturer part#"
 	1    2500 5100
 	1    0    0    -1
@@
 F 0 "R5" H 2268 5146 50  0000 L CNN
 F 1 "4.7K" H 2268 5055 50  0000 L CNN
-F 2 "Resistor_THT:R_Axial_DIN0207_L6.3mm_D2.5mm_P10.16mm_Horizontal" H 2200 5100 50  0001 C CNN
-F 3 "https://www.seielect.com/catalog/sei-cf_cfm.pdf" H 2200 5100 50  0001 C CNN
-F 4 "digikey" H 2200 5100 50  0001 C CNN "Vendor"
-F 5 "CF14JT4K70CT-ND  " H 2200 5100 50  0001 C CNN "Vendor part#"
-F 6 "Stackpole Electronics Inc" H 2200 5100 50  0001 C CNN "Manufacturer part#"
+F 2 "Resistor_SMD:R_1206_3216Metric_Pad1.30x1.75mm_HandSolder" H 2200 5100 50  0001 C CNN
+F 3 "https://datasheet.lcsc.com/lcsc/1810301414_UNI-ROYAL-Uniroyal-Elec-1206W4F4701T5E_C17936.pdf" H 2200 5100 50  0001 C CNN
+F 4 "JLCPCB" H 2200 5100 50  0001 C CNN "Vendor"
+F 5 "C17936" H 2200 5100 50  0001 C CNN "Vendor part#"
+F 6 "1206W4F4701T5E" H 2200 5100 50  0001 C CNN "Manufacturer part#"
 	1    2200 5100
 	1    0    0    -1
@@
 F 0 "C3" H 1738 4746 50  0000 L CNN
 F 1 "1uF 50V" H 1738 4655 50  0000 L CNN
-F 2 "Capacitor_THT:CP_Radial_D5.0mm_P2.00mm" H 1650 4700 50  0001 C CNN
-F 3 "https://www.vishay.com/docs/42052/515d.pdf" H 1650 4700 50  0001 C CNN
-F 4 "digikey" H 1650 4700 50  0001 C CNN "Vendor"
-F 5 "718-2229-ND" H 1650 4700 50  0001 C CNN "Vendor part#"
-F 6 "515D105M050JA6AE3" H 1650 4700 50  0001 C CNN "Manufacturer part#"
+F 2 "Capacitor_SMD:CP_Elec_4x5.4" H 1650 4700 50  0001 C CNN
+F 3 " https://datasheet.lcsc.com/lcsc/2105211834_Honor-Elec-RVT1H1R0M0405_C3348.pdf" H 1650 4700 50  0001 C CNN
+F 4 "JLCPCB" H 1650 4700 50  0001 C CNN "Vendor"
+F 5 "C3348" H 1650 4700 50  0001 C CNN "Vendor part#"
+F 6 "RVT1H1R0M0405" H 1650 4700 50  0001 C CNN "Manufacturer part#"
 	1    1650 4700
 	1    0    0    -1
@@
 F 0 "C2" V 6125 3600 50  0000 C CNN
 F 1 "10uF 25v" V 6034 3600 50  0000 C CNN
-F 2 "Capacitor_THT:CP_Radial_D5.0mm_P2.00mm" H 5900 3600 50  0001 C CNN
-F 3 "http://nichicon-us.com/english/products/pdfs/e-upw.pdf" H 5900 3600 50  0001 C CNN
-F 4 "digikey" V 5900 3600 50  0001 C CNN "Vendor"
-F 5 "493-1809-ND" V 5900 3600 50  0001 C CNN "Vendor part#"
-F 6 "UPW1E100MDD" V 5900 3600 50  0001 C CNN "Manufacturer part#"
+F 2 "Capacitor_SMD:CP_Elec_4x5.3" H 5900 3600 50  0001 C CNN
+F 3 "https://datasheet.lcsc.com/lcsc/1809291326_Lelon-VE-100M1ETR-0405_C134721.pdf" H 5900 3600 50  0001 C CNN
+F 4 "JLCPCB" V 5900 3600 50  0001 C CNN "Vendor"
+F 5 "C134721" V 5900 3600 50  0001 C CNN "Vendor part#"
+F 6 "VE-100M1ETR-0405" V 5900 3600 50  0001 C CNN "Manufacturer part#"
 	1    5900 3600
 	0    -1   -1   0
@@
 F 0 "IC3" H 3400 2720 50  0000 C CNN
 F 1 "SN74LS245N" H 3400 2629 50  0000 C CNN
-F 2 "Package_DIP:DIP-20_W7.62mm_Socket" H 3000 2900 50  0001 L BNN
-F 3 "https://www.ti.com/lit/ds/sdls146b/sdls146b.pdf" H 3400 1750 50  0001 L BNN
-F 4 "digikey" H 3400 1750 50  0001 C CNN "Vendor"
-F 5 "296-1655-5-ND" H 3400 1750 50  0001 C CNN "Vendor part#"
-F 6 "SN74LS245N" H 3400 1750 50  0001 C CNN "Manufacturer part#"
+F 2 "Package_SO:SOIC-20W_7.5x12.8mm_P1.27mm" H 3000 2900 50  0001 L BNN
+F 3 "https://datasheet.lcsc.com/lcsc/1810010228_Texas-Instruments-SN74LS245DWR_C129580.pdf" H 3400 1750 50  0001 L BNN
+F 4 "JLCPCB" H 3400 1750 50  0001 C CNN "Vendor"
+F 5 "C129580" H 3400 1750 50  0001 C CNN "Vendor part#"
+F 6 "SN74LS245DWR" H 3400 1750 50  0001 C CNN "Manufacturer part#"
 	1    3400 1750
 	1    0    0    -1
@@
 F 0 "C5" V 2071 1000 50  0000 C CNN
 F 1 ".033uF" V 2162 1000 50  0000 C CNN
-F 2 "Capacitor_THT:C_Axial_L5.1mm_D3.1mm_P10.00mm_Horizontal" H 2300 1000 50  0001 C CNN
-F 3 "https://api.kemet.com/component-edge/download/datasheet/C410C333K5R5TA7200.pdf" H 2300 1000 50  0001 C CNN
-F 4 "digikey" H 2300 1000 50  0001 C CNN "Vendor"
-F 5 "399-4470-1-ND" H 2300 1000 50  0001 C CNN "Vendor part#"
-F 6 "C410C333K5R5TA7200" H 2300 1000 50  0001 C CNN "Manufacturer part#"
+F 2 "Capacitor_SMD:C_0805_2012Metric_Pad1.18x1.45mm_HandSolder" H 2300 1000 50  0001 C CNN
+F 3 "https://datasheet.lcsc.com/lcsc/1811061723_FH-Guangdong-Fenghua-Advanced-Tech-0805B333K500NT_C1739.pdf" H 2300 1000 50  0001 C CNN
+F 4 "JLCPCB" H 2300 1000 50  0001 C CNN "Vendor"
+F 5 "C1739" H 2300 1000 50  0001 C CNN "Vendor part#"
+F 6 "0805B333K500NT" H 2300 1000 50  0001 C CNN "Manufacturer part#"
 	1    2300 1000
 	0    1    1    0

Commit message: -converted more components from THT to SMD -replaced SALT chip with replacement circuitry
Parts:
- D12: footprint Diode_THT:D_DO-35_SOD27_P7.62mm_Horizontal -> Diode_SMD:D_SOD-323F; Manufacturer part# 1N4148 -> 1N4148WS; Vendor digikey -> JLCPCB; Vendor part# 1N4148FS-ND -> C2128
- R1: footprint Resistor_THT:R_Axial_DIN0207_L6.3mm_D2.5mm_P10.16mm_Horizontal -> Resistor_SMD:R_1206_3216Metric_Pad1.30x1.75mm_HandSolder; Manufacturer part# MFR-25FBF52-100K -> 1206W4F1003T5E; Vendor digikey -> JLCPCB; Vendor part# 100KXBK-ND -> C17900
Changed lines of the file:
@@
 F 0 "D12" V 1950 3950 50  0000 L CNN
 F 1 "1N4148" V 2100 3900 50  0000 L CNN
-F 2 "Diode_THT:D_DO-35_SOD27_P7.62mm_Horizontal" H 2050 4075 50  0001 C CNN
-F 3 " https://www.onsemi.com/pub/Collateral/1N914-D.PDF" H 2050 4250 50  0001 C CNN
-F 4 "digikey" V 2050 4250 50  0001 C CNN "Vendor"
-F 5 "1N4148FS-ND" V 2050 4250 50  0001 C CNN "Vendor part#"
-F 6 "1N4148" V 2050 4250 50  0001 C CNN "Manufacturer part#"
+F 2 "Diode_SMD:D_SOD-323F" H 2050 4075 50  0001 C CNN
+F 3 "https://datasheet.lcsc.com/lcsc/1810101110_Changjiang-Electronics-Tech--CJ-1N4148WS_C2128.pdf" H 2050 4250 50  0001 C CNN
+F 4 "JLCPCB" V 2050 4250 50  0001 C CNN "Vendor"
+F 5 "C2128" V 2050 4250 50  0001 C CNN "Vendor part#"
+F 6 "1N4148WS" V 2050 4250 50  0001 C CNN "Manufacturer part#"
 	1    2050 4250
 	0    -1   1    0
@@
 F 0 "R1" H 1718 4346 50  0000 L CNN
 F 1 "100K" H 1718 4255 50  0000 L CNN
-F 2 "Resistor_THT:R_Axial_DIN0207_L6.3mm_D2.5mm_P10.16mm_Horizontal" H 1650 4300 50  0001 C CNN
-F 3 "https://www.yageo.com/upload/media/product/products/datasheet/lr/Yageo_LR_MFR_1.pdf" H 1650 4300 50  0001 C CNN
-F 4 "digikey" H 1650 4300 50  0001 C CNN "Vendor"
-F 5 "100KXBK-ND" H 1650 4300 50  0001 C CNN "Vendor part#"
-F 6 "MFR-25FBF52-100K" H 1650 4300 50  0001 C CNN "Manufacturer part#"
+F 2 "Resistor_SMD:R_1206_3216Metric_Pad1.30x1.75mm_HandSolder" H 1650 4300 50  0001 C CNN
+F 3 " https://datasheet.lcsc.com/lcsc/1810301421_UNI-ROYAL-Uniroyal-Elec-1206W4F1003T5E_C17900.pdf" H 1650 4300 50  0001 C CNN
+F 4 "JLCPCB" H 1650 4300 50  0001 C CNN "Vendor"
+F 5 "C17900" H 1650 4300 50  0001 C CNN "Vendor part#"
+F 6 "1206W4F1003T5E" H 1650 4300 50  0001 C CNN "Manufacturer part#"
 	1    1650 4300
 	-1   0    0    -1

Commit message: routed the board
Parts:
- C2: value 10uF 25v -> 10uF 16v; footprint Capacitor_SMD:CP_Elec_4x5.3 -> Capacitor_Tantalum_SMD:CP_EIA-3216-18_Kemet-A; Manufacturer part# VE-100M1ETR-0405 -> TAJA106K016RNJ; Vendor part# C134721 -> C7171
- C3: value 1uF 50V -> 10uF 16v; footprint Capacitor_SMD:CP_Elec_4x5.4 -> Capacitor_Tantalum_SMD:CP_EIA-3216-18_Kemet-A; Manufacturer part# RVT1H1R0M0405 -> TAJA106K016RNJ; Vendor part# C3348 -> C7171
Connections:
- net GNDS: no longer IC3.19 (~OE)
- net BUS_TXRX_ENABLE: now reaches IC1.6 (BA)
- net BUS_TXRX_ENABLE: now also IC3.19 (~OE)
- no-connect marks 5 -> 4
Changed lines of the file:
@@
 $EndComp
 NoConn ~ 5800 6550
-NoConn ~ 5800 6450
 NoConn ~ 5800 6150
 NoConn ~ 5800 6050
@@
 	1    0    0    -1
 $EndComp
-Wire Wire Line
-	5300 6950 5300 7100
 $Comp
 L power:+5V #PWR01027
@@
 	2700 2350 2450 2350
 Wire Wire Line
-	5800 6350 6100 6350
-Wire Wire Line
-	6100 6350 6100 7100
-Wire Wire Line
-	6100 7100 5300 7100
-Connection ~ 5300 7100
-Wire Wire Line
 	4800 5250 4300 5250
 Wire Wire Line
@@
 AR Path="/60273794/60456BFE" Ref="C3"  Part="1"
 F 0 "C3" H 1738 4746 50  0000 L CNN
-F 1 "1uF 50V" H 1738 4655 50  0000 L CNN
-F 2 "Capacitor_SMD:CP_Elec_4x5.4" H 1650 4700 50  0001 C CNN
-F 3 " https://datasheet.lcsc.com/lcsc/2105211834_Honor-Elec-RVT1H1R0M0405_C3348.pdf" H 1650 4700 50  0001 C CNN
+F 1 "10uF 16v" H 1738 4655 50  0000 L CNN
+F 2 "Capacitor_Tantalum_SMD:CP_EIA-3216-18_Kemet-A" H 1650 4700 50  0001 C CNN
+F 3 "https://datasheet.lcsc.com/lcsc/1811071223_AVX-TAJA106K016RNJ_C7171.pdf" H 1650 4700 50  0001 C CNN
 F 4 "JLCPCB" H 1650 4700 50  0001 C CNN "Vendor"
-F 5 "C3348" H 1650 4700 50  0001 C CNN "Vendor part#"
-F 6 "RVT1H1R0M0405" H 1650 4700 50  0001 C CNN "Manufacturer part#"
+F 5 "C7171" H 1650 4700 50  0001 C CNN "Vendor part#"
+F 6 "TAJA106K016RNJ" H 1650 4700 50  0001 C CNN "Manufacturer part#"
 	1    1650 4700
 	1    0    0    -1
@@
 P 5900 3600
 F 0 "C2" V 6125 3600 50  0000 C CNN
-F 1 "10uF 25v" V 6034 3600 50  0000 C CNN
-F 2 "Capacitor_SMD:CP_Elec_4x5.3" H 5900 3600 50  0001 C CNN
-F 3 "https://datasheet.lcsc.com/lcsc/1809291326_Lelon-VE-100M1ETR-0405_C134721.pdf" H 5900 3600 50  0001 C CNN
+F 1 "10uF 16v" V 6034 3600 50  0000 C CNN
+F 2 "Capacitor_Tantalum_SMD:CP_EIA-3216-18_Kemet-A" H 5900 3600 50  0001 C CNN
+F 3 "https://datasheet.lcsc.com/lcsc/1811071223_AVX-TAJA106K016RNJ_C7171.pdf" H 5900 3600 50  0001 C CNN
 F 4 "JLCPCB" V 5900 3600 50  0001 C CNN "Vendor"
-F 5 "C134721" V 5900 3600 50  0001 C CNN "Vendor part#"
-F 6 "VE-100M1ETR-0405" V 5900 3600 50  0001 C CNN "Manufacturer part#"
+F 5 "C7171" V 5900 3600 50  0001 C CNN "Vendor part#"
+F 6 "TAJA106K016RNJ" V 5900 3600 50  0001 C CNN "Manufacturer part#"
 	1    5900 3600
 	0    -1   -1   0
@@
 	2950 6550 4800 6550
 Wire Wire Line
-	5300 7100 5300 7550
-Wire Wire Line
 	2950 6650 4800 6650
 $Comp
@@
 L power:GNDS #PWR01024
 U 1 1 61507CAC
-P 1950 1500
-F 0 "#PWR01024" H 1950 1250 50  0001 C CNN
-F 1 "GNDS" H 1955 1327 50  0000 C CNN
-F 2 "" H 1950 1500 50  0001 C CNN
-F 3 "" H 1950 1500 50  0001 C CNN
-	1    1950 1500
-	1    0    0    -1
-$EndComp
-Wire Wire Line
-	2700 1350 1950 1350
+P 1550 1500
+F 0 "#PWR01024" H 1550 1250 50  0001 C CNN
+F 1 "GNDS" H 1555 1327 50  0000 C CNN
+F 2 "" H 1550 1500 50  0001 C CNN
+F 3 "" H 1550 1500 50  0001 C CNN
+	1    1550 1500
+	1    0    0    -1
+$EndComp
 $Comp
 L Device:C_Small C?
@@
 $EndComp
 Wire Wire Line
-	2200 1000 1950 1000
-Wire Wire Line
-	1950 1000 1950 1350
-Connection ~ 1950 1350
-Wire Wire Line
-	1950 1350 1950 1500
-Wire Wire Line
 	2400 1000 2550 1000
 Connection ~ 2550 1000
@@
 Wire Wire Line
 	1150 4500 1650 4500
+Wire Wire Line
+	1550 1000 1550 1500
+Text Label 5950 6450 0    50   ~ 0
+BUS_TXRX_ENABLE
+Wire Wire Line
+	5950 6450 5800 6450
+Wire Wire Line
+	5300 6950 5300 7550
+$Comp
+L power:GNDS #PWR0106
+U 1 1 6199B2E5
+P 7150 6500
+F 0 "#PWR0106" H 7150 6250 50  0001 C CNN
+F 1 "GNDS" H 7155 6327 50  0000 C CNN
+F 2 "" H 7150 6500 50  0001 C CNN
+F 3 "" H 7150 6500 50  0001 C CNN
+	1    7150 6500
+	1    0    0    -1
+$EndComp
+Wire Wire Line
+	7150 6350 7150 6500
+Wire Wire Line
+	5800 6350 7150 6350
+Text Label 2600 1350 2    50   ~ 0
+BUS_TXRX_ENABLE
+Wire Wire Line
+	1550 1000 2200 1000
+Wire Wire Line
+	2700 1350 2600 1350
 Wire Bus Line
 	2350 1750 2350 2450
