File: coco3/gime.sch (KiCad schematic (older format))
At the start: 39 parts, among them IC10 74LS244, IC11 74LS244, IC12 74LS244, IC13 74LS374, IC15 74LS04, IC6 TCC1014, IC9 74LS138, X1 28.63636 MHz

Commit message: -replaced PIA's with he PLCC44 package versions -removed RF modulator -removed DRAM
Parts:
- removed C65: 82pF, Capacitor_THT:C_Rect_L7.2mm_W3.0mm_P5.00mm_FKS2_FKP2_MKS2_MKP2, symbol Device:C_Small
- removed C66: 27pF, Capacitor_THT:C_Rect_L7.2mm_W3.0mm_P5.00mm_FKS2_FKP2_MKS2_MKP2, symbol Device:C_Small
- removed JP65, JP66: SolderJumper_2_Open, Jumper:SolderJumper-2_P1.3mm_Open_RoundedPad1.0x1.5mm, symbol Jumper:SolderJumper_2_Open
Connections:
- wire segments 292 -> 285
Changed lines of the file:
@@
 Wire Wire Line
 	6000 5550 6000 5650
-$Comp
-L Device:C_Small C?
-U 1 1 6136F6EC
-P 6000 6400
-AR Path="/60273794/6136F6EC" Ref="C?"  Part="1"
-AR Path="/602A51A8/6136F6EC" Ref="C?"  Part="1"
-AR Path="/603CF7B8/6136F6EC" Ref="C?"  Part="1"
-AR Path="/61257512/6136F6EC" Ref="C66"  Part="1"
-F 0 "C66" H 5850 6400 50  0000 C CNN
-F 1 "27pF" H 5850 6500 50  0000 C CNN
-F 2 "Capacitor_THT:C_Rect_L7.2mm_W3.0mm_P5.00mm_FKS2_FKP2_MKS2_MKP2" H 6000 6400 50  0001 C CNN
-F 3 "https://www.vishay.com/docs/45171/kseries.pdf" H 6000 6400 50  0001 C CNN
-F 4 "digikey" V 6000 6400 50  0001 C CNN "Vendor"
-F 5 "BC1035CT-ND" V 6000 6400 50  0001 C CNN "Vendor part#"
-F 6 "K270J15C0GF5TH5" V 6000 6400 50  0001 C CNN "Manufacturer part#"
-	1    6000 6400
-	-1   0    0    1
-$EndComp
-$Comp
-L Device:C_Small C?
-U 1 1 6138ACD5
-P 5850 6400
-AR Path="/60273794/6138ACD5" Ref="C?"  Part="1"
-AR Path="/602A51A8/6138ACD5" Ref="C?"  Part="1"
-AR Path="/603CF7B8/6138ACD5" Ref="C?"  Part="1"
-AR Path="/61257512/6138ACD5" Ref="C65"  Part="1"
-F 0 "C65" H 5700 6400 50  0000 C CNN
-F 1 "82pF" H 5700 6500 50  0000 C CNN
-F 2 "Capacitor_THT:C_Rect_L7.2mm_W3.0mm_P5.00mm_FKS2_FKP2_MKS2_MKP2" H 5850 6400 50  0001 C CNN
-F 3 "https://www.vishay.com/docs/45171/kseries.pdf" H 5850 6400 50  0001 C CNN
-F 4 "digikey" V 5850 6400 50  0001 C CNN "Vendor"
-F 5 "BC1041CT-ND" V 5850 6400 50  0001 C CNN "Vendor part#"
-F 6 "K820J15C0GF5TH5" V 5850 6400 50  0001 C CNN "Manufacturer part#"
-	1    5850 6400
-	1    0    0    1
-$EndComp
-$Comp
-L power:GNDS #PWR?
-U 1 1 6138FA4F
-P 5950 6650
-AR Path="/602A51A8/6138FA4F" Ref="#PWR?"  Part="1"
-AR Path="/60308A73/6138FA4F" Ref="#PWR?"  Part="1"
-AR Path="/603E4732/6138FA4F" Ref="#PWR?"  Part="1"
-AR Path="/603D345E/6138FA4F" Ref="#PWR?"  Part="1"
-AR Path="/6138FA4F" Ref="#PWR?"  Part="1"
-AR Path="/61257512/6138FA4F" Ref="#PWR0101"  Part="1"
-F 0 "#PWR0101" H 5950 6400 50  0001 C CNN
-F 1 "GNDS" H 5950 6500 50  0000 C CNN
-F 2 "" H 5950 6650 50  0001 C CNN
-F 3 "" H 5950 6650 50  0001 C CNN
-	1    5950 6650
-	-1   0    0    -1
-$EndComp
-Wire Wire Line
-	5850 6500 5850 6550
-Wire Wire Line
-	5850 6550 5950 6550
-Wire Wire Line
-	5950 6550 5950 6650
-Wire Wire Line
-	6000 6500 6000 6550
-Wire Wire Line
-	6000 6550 5950 6550
-Connection ~ 5950 6550
 Wire Wire Line
 	6000 5850 6000 5950
@@
 Wire Wire Line
 	5650 5950 5850 5950
-Connection ~ 5850 5950
-Wire Wire Line
-	5850 5950 5850 6000
 Wire Wire Line
 	6200 5950 6150 5950
-Connection ~ 6000 5950
-Wire Wire Line
-	6000 5950 6000 6000
 $Comp
 L Connector:TestPoint TP?
@@
 Wire Wire Line
 	10550 5000 10550 5200
-$Comp
-L Jumper:SolderJumper_2_Open JP65
-U 1 1 61321980
-P 5850 6150
-F 0 "JP65" V 5850 5900 50  0000 L CNN
-F 1 "SolderJumper_2_Open" V 5895 6218 50  0001 L CNN
-F 2 "Jumper:SolderJumper-2_P1.3mm_Open_RoundedPad1.0x1.5mm" H 5850 6150 50  0001 C CNN
-F 3 "~" H 5850 6150 50  0001 C CNN
-	1    5850 6150
-	0    1    1    0
-$EndComp
-$Comp
-L Jumper:SolderJumper_2_Open JP66
-U 1 1 61359175
-P 6000 6150
-F 0 "JP66" V 6000 6250 50  0000 L CNN
-F 1 "SolderJumper_2_Open" V 6045 6218 50  0001 L CNN
-F 2 "Jumper:SolderJumper-2_P1.3mm_Open_RoundedPad1.0x1.5mm" H 6000 6150 50  0001 C CNN
-F 3 "~" H 6000 6150 50  0001 C CNN
-	1    6000 6150
-	0    1    1    0
-$EndComp
 Wire Bus Line
 	3650 4850 3650 6950

Commit message: -repplaced a whole bunch of THT components with SMT components
Parts:
- C10, C11: footprint Capacitor_THT:C_Disc_D4.7mm_W2.5mm_P5.00mm -> Capacitor_SMD:C_0805_2012Metric_Pad1.18x1.45mm_HandSolder; Manufacturer part# K390J15C0GF5TL2 -> 0805N390J500CT; Vendor digikey -> JLCPCB; Vendor part# BC1008CT-ND -> C296098
- C12, C38, C39, C40, C41, C8: footprint Capacitor_THT:C_Disc_D4.7mm_W2.5mm_P5.00mm -> Capacitor_SMD:C_0805_2012Metric_Pad1.18x1.45mm_HandSolder; Manufacturer part# FG28C0G1H103JNT06 -> CL21A106KAYNNNE; Vendor digikey -> JLCPCB; Vendor part# 445-173474-1-ND -> C15850
- C60: footprint Capacitor_THT:C_Rect_L7.2mm_W3.0mm_P5.00mm_FKS2_FKP2_MKS2_MKP2 -> Capacitor_SMD:C_0805_2012Metric_Pad1.18x1.45mm_HandSolder; Manufacturer part# FA28NP01H330JNU06 -> CL21C330JBANNNC; Vendor digikey -> JLCPCB; Vendor part# 445-180775-1-ND -> C1814
- C64: footprint Capacitor_THT:C_Rect_L7.2mm_W2.5mm_P5.00mm_FKS2_FKP2_MKS2_MKP2 -> Capacitor_SMD:C_0805_2012Metric_Pad1.18x1.45mm_HandSolder; Manufacturer part# FA28C0G2E151JNU06 -> 0805B151K500NT; Vendor digikey -> JLCPCB; Vendor part# 445-180756-1-ND -> C1716
- C9: footprint Capacitor_THT:CP_Radial_D5.0mm_P2.00mm -> Capacitor_SMD:CP_Elec_6.3x5.3; Manufacturer part# 16ZLH100MEFC5X11 -> VEJ101M1CTR-0605; Vendor digikey -> JLCPCB; Vendor part# 1189-1148-ND -> C164064
- IC10, IC11, IC12: footprint Package_DIP:DIP-20_W7.62mm_Socket -> Package_SO:SOIC-20W_7.5x12.8mm_P1.27mm; Manufacturer part# SN74LS244N -> SN74LS244DWR; Vendor digikey -> JLCPCB; Vendor part# 296-1653-5-ND -> C7751
- IC13: footprint Package_DIP:DIP-20_W7.62mm_Socket -> Package_SO:SOIC-20W_7.5x12.8mm_P1.27mm; Manufacturer part# SN74ALS374AN -> SN74LS374NSR; Vendor digikey -> JLCPCB; Vendor part# 296-1498-5-ND -> C7764
- IC15: footprint Package_DIP:DIP-14_W7.62mm_Socket -> Package_SO:SOIC-14_3.9x8.7mm_P1.27mm; Manufacturer part# SN74LS04N -> SN74LS04DR; Vendor digikey -> JLCPCB; Vendor part# 296-1629-5-ND -> C6796
- IC9: footprint Package_DIP:DIP-16_W7.62mm_Socket -> Package_SO:SOP-16_3.9x9.9mm_P1.27mm; Manufacturer part# SN74LS138N -> XL74LS138; Vendor digikey -> JLCPCB; Vendor part# 296-1639-5-ND -> C513515
- R11, R8: footprint Resistor_THT:R_Axial_DIN0207_L6.3mm_D2.5mm_P10.16mm_Horizontal -> Resistor_SMD:R_1206_3216Metric_Pad1.30x1.75mm_HandSolder; Manufacturer part# Stackpole Electronics Inc -> 1206W4F4701T5E; Vendor digikey -> JLCPCB; Vendor part# CF14JT4K70CT-ND -> C17936
- R22: footprint Resistor_THT:R_Axial_DIN0207_L6.3mm_D2.5mm_P10.16mm_Horizontal -> Resistor_SMD:R_1206_3216Metric_Pad1.30x1.75mm_HandSolder; Manufacturer part# CF14JT120R -> 1206W4F1200T5E; Vendor digikey -> JLCPCB; Vendor part# CF14JT120RCT-ND -> C17909

Commit message: -converted more components from THT to SMD -replaced SALT chip with replacement circuitry
Parts:
- R10, R9: footprint Resistor_THT:R_Axial_DIN0309_L9.0mm_D3.2mm_P12.70mm_Horizontal -> Resistor_SMD:R_1206_3216Metric_Pad1.30x1.75mm_HandSolder; Manufacturer part# CF12JT47R0 -> 1206W4J0470T5E; Vendor digikey -> JLCPCB; Vendor part# CF12JT47R0CT-ND -> C25384
- R23: footprint Resistor_THT:R_Axial_DIN0207_L6.3mm_D2.5mm_P10.16mm_Horizontal -> Resistor_SMD:R_1206_3216Metric_Pad1.30x1.75mm_HandSolder; Manufacturer part# CF1/4CT52R820J -> 1206W4F820JT5E; Vendor digikey -> JLCPCB; Vendor part# 2019-CF1/4CT52R820JCT-ND -> C17980
- R63: footprint Resistor_THT:R_Axial_DIN0309_L9.0mm_D3.2mm_P12.70mm_Horizontal -> Resistor_SMD:R_1206_3216Metric_Pad1.30x1.75mm_HandSolder; Manufacturer part# CF12JT150R -> 1206W4F1500T5E; Vendor digikey -> JLCPCB; Vendor part# CF12JT150RCT-ND -> C17917
- R65: footprint Resistor_THT:R_Axial_DIN0207_L6.3mm_D2.5mm_P10.16mm_Horizontal -> Resistor_SMD:R_1206_3216Metric_Pad1.30x1.75mm_HandSolder; Manufacturer part# RNF14FTD1M00 -> 1206W4F1004T5E; Vendor digikey -> JLCPCB; Vendor part# RNF14FTD1M00CT-ND -> C17927
Changed lines of the file:
@@
 F 0 "R9" V 9950 4700 50  0000 L CNN
 F 1 "47" V 9850 4850 50  0000 L CNN
-F 2 "Resistor_THT:R_Axial_DIN0309_L9.0mm_D3.2mm_P12.70mm_Horizontal" H 9900 4800 50  0001 C CNN
-F 3 "https://www.seielect.com/catalog/sei-cf_cfm.pdf" H 9900 4800 50  0001 C CNN
-F 4 "digikey" H 9900 4800 50  0001 C CNN "Vendor"
-F 5 "CF12JT47R0CT-ND" H 9900 4800 50  0001 C CNN "Vendor part#"
-F 6 "CF12JT47R0" H 9900 4800 50  0001 C CNN "Manufacturer part#"
+F 2 "Resistor_SMD:R_1206_3216Metric_Pad1.30x1.75mm_HandSolder" H 9900 4800 50  0001 C CNN
+F 3 "https://datasheet.lcsc.com/lcsc/1811101020_UNI-ROYAL-Uniroyal-Elec-1206W4J0470T5E_C25384.pdf" H 9900 4800 50  0001 C CNN
+F 4 "JLCPCB" H 9900 4800 50  0001 C CNN "Vendor"
+F 5 "C25384" H 9900 4800 50  0001 C CNN "Vendor part#"
+F 6 "1206W4J0470T5E" H 9900 4800 50  0001 C CNN "Manufacturer part#"
 	1    9900 4800
 	0    1    -1   0
@@
 F 0 "R10" V 9950 4850 50  0000 L CNN
 F 1 "47" V 9850 5000 50  0000 L CNN
-F 2 "Resistor_THT:R_Axial_DIN0309_L9.0mm_D3.2mm_P12.70mm_Horizontal" H 9900 4950 50  0001 C CNN
-F 3 "https://www.seielect.com/catalog/sei-cf_cfm.pdf" H 9900 4950 50  0001 C CNN
-F 4 "digikey" H 9900 4950 50  0001 C CNN "Vendor"
-F 5 "CF12JT47R0CT-ND" H 9900 4950 50  0001 C CNN "Vendor part#"
-F 6 "CF12JT47R0" H 9900 4950 50  0001 C CNN "Manufacturer part#"
+F 2 "Resistor_SMD:R_1206_3216Metric_Pad1.30x1.75mm_HandSolder" H 9900 4950 50  0001 C CNN
+F 3 "https://datasheet.lcsc.com/lcsc/1811101020_UNI-ROYAL-Uniroyal-Elec-1206W4J0470T5E_C25384.pdf" H 9900 4950 50  0001 C CNN
+F 4 "JLCPCB" H 9900 4950 50  0001 C CNN "Vendor"
+F 5 "C25384" H 9900 4950 50  0001 C CNN "Vendor part#"
+F 6 "1206W4J0470T5E" H 9900 4950 50  0001 C CNN "Manufacturer part#"
 	1    9900 4950
 	0    1    -1   0
@@
 F 0 "R63" H 7750 5800 50  0000 L CNN
 F 1 "150" H 7700 5700 50  0000 L CNN
-F 2 "Resistor_THT:R_Axial_DIN0309_L9.0mm_D3.2mm_P12.70mm_Horizontal" H 7900 5700 50  0001 C CNN
-F 3 "https://www.seielect.com/catalog/sei-cf_cfm.pdf" H 7900 5700 50  0001 C CNN
-F 4 "digikey" H 7900 5700 50  0001 C CNN "Vendor"
-F 5 "CF12JT150RCT-ND" H 7900 5700 50  0001 C CNN "Vendor part#"
-F 6 "CF12JT150R" H 7900 5700 50  0001 C CNN "Manufacturer part#"
+F 2 "Resistor_SMD:R_1206_3216Metric_Pad1.30x1.75mm_HandSolder" H 7900 5700 50  0001 C CNN
+F 3 "https://datasheet.lcsc.com/lcsc/1809140241_UNI-ROYAL-Uniroyal-Elec-1206W4F1500T5E_C17917.pdf" H 7900 5700 50  0001 C CNN
+F 4 "JLCPCB" H 7900 5700 50  0001 C CNN "Vendor"
+F 5 "C17917" H 7900 5700 50  0001 C CNN "Vendor part#"
+F 6 "1206W4F1500T5E" H 7900 5700 50  0001 C CNN "Manufacturer part#"
 	1    7900 5700
 	-1   0    0    -1
@@
 F 0 "R65" V 8550 5750 50  0000 L CNN
 F 1 "1M" V 8300 5700 50  0000 L CNN
-F 2 "Resistor_THT:R_Axial_DIN0207_L6.3mm_D2.5mm_P10.16mm_Horizontal" H 8400 5900 50  0001 C CNN
-F 3 "  https://www.seielect.com/catalog/sei-rnf_rnmf.pdf" H 8400 5900 50  0001 C CNN
-F 4 "digikey" H 8400 5900 50  0001 C CNN "Vendor"
-F 5 "RNF14FTD1M00CT-ND" H 8400 5900 50  0001 C CNN "Vendor part#"
-F 6 "RNF14FTD1M00" H 8400 5900 50  0001 C CNN "Manufacturer part#"
+F 2 "Resistor_SMD:R_1206_3216Metric_Pad1.30x1.75mm_HandSolder" H 8400 5900 50  0001 C CNN
+F 3 " https://datasheet.lcsc.com/lcsc/1811050105_UNI-ROYAL-Uniroyal-Elec-1206W4F1004T5E_C17927.pdf" H 8400 5900 50  0001 C CNN
+F 4 "JLCPCB" H 8400 5900 50  0001 C CNN "Vendor"
+F 5 "C17927" H 8400 5900 50  0001 C CNN "Vendor part#"
+F 6 "1206W4F1004T5E" H 8400 5900 50  0001 C CNN "Manufacturer part#"
 	1    8400 5900
 	0    1    -1   0
@@
 F 0 "R23" H 5800 5700 50  0000 L CNN
 F 1 "82" H 5800 5800 50  0000 L CNN
-F 2 "Resistor_THT:R_Axial_DIN0207_L6.3mm_D2.5mm_P10.16mm_Horizontal" H 6000 5750 50  0001 C CNN
-F 3 "https://www.koaspeer.com/pdfs/CF.pdf" H 6000 5750 50  0001 C CNN
-F 4 "digikey" H 6000 5750 50  0001 C CNN "Vendor"
-F 5 "2019-CF1/4CT52R820JCT-ND" H 6000 5750 50  0001 C CNN "Vendor part#"
-F 6 "CF1/4CT52R820J" H 6000 5750 50  0001 C CNN "Manufacturer part#"
+F 2 "Resistor_SMD:R_1206_3216Metric_Pad1.30x1.75mm_HandSolder" H 6000 5750 50  0001 C CNN
+F 3 "https://datasheet.lcsc.com/lcsc/1810301412_UNI-ROYAL-Uniroyal-Elec-1206W4F820JT5E_C17980.pdf" H 6000 5750 50  0001 C CNN
+F 4 "JLCPCB" H 6000 5750 50  0001 C CNN "Vendor"
+F 5 "C17980" H 6000 5750 50  0001 C CNN "Vendor part#"
+F 6 "1206W4F820JT5E" H 6000 5750 50  0001 C CNN "Manufacturer part#"
 	1    6000 5750
 	-1   0    0    1
